File: example/pcb/pcb.kicad_sch (KiCad schematic)
At the start: 10 parts, among them IC1 AD8403ARUZ1-REEL, IC2 AD8403ARUZ1-REEL, J1 Conn_01x06_Pin, J2 Conn_01x06_Pin, J3 Conn_01x05_Pin

Commit message: Update pcb
Parts:
- removed C2: 100n, Capacitor_SMD:C_0603_1608Metric, symbol Device:C_Small
- removed IC2: AD8403ARUZ1-REEL, AD8403ARUZ1-REEL:SOP65P640X120-24N, symbol AD8403ARUZ1-REEL:AD8403ARUZ1-REEL
- removed J3: Conn_01x05_Pin, Connector_PinHeader_2.54mm:PinHeader_1x05_P2.54mm_Vertical, symbol Connector:Conn_01x05_Pin
- removed R3: 10k, Resistor_SMD:R_0603_1608Metric, symbol Device:R_Small
Connections:
- net RS_2 is gone; now on net SDO: J2.6 (Pin_6)
- net SHDN_2 is gone; now on net SDI: J2.5 (Pin_5)
- net W1_2 is gone; now on net GND: J2.1 (Pin_1)
- net W2_2 is gone; now on net +3V3: J2.2 (Pin_2)
- net W3_2 is gone; now on net CS: J2.3 (Pin_3)
- net W4_2 is gone; now on net CLK: J2.4 (Pin_4)
- net SDO: now reaches IC1.13 (SDO), R1.2
- net RS_1 renamed RS
- net RS: now also J1.5 (Pin_5); no longer J1.6 (Pin_6)
- net SHDN_1 renamed SHDN
- net SHDN: now also J1.6 (Pin_6); no longer J1.5 (Pin_5)
- net W1_1 renamed W1
- net W2_1 renamed W2
- net W3_1 renamed W3
- net W4_1 renamed W4
